File: eagle/scifair/sci fair schematic.sch (EAGLE design)
At the start: 19 parts, among them IC1 LM555N, IC2 LM340H-12, Q1 BC817-16W, Q2 BC817-16W, X1 RIGHT, X2 LEFT, X3 PWR

Commit message: Add a space using vias for jumpers to go to a rocker switch
Connections:
- net N$5 renamed GND
Changed lines of the file:
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@@
 </segment>
 </net>
-<net name="N$5" class="0">
+<net name="GND" class="0">
 <segment>
 <pinref part="X3" gate="G$1" pin="4"/>
