File: eagle/scifair/sci fair schematic.sch (EAGLE design)
At the start: 16 parts, among them IC1 LM555N, IC2 LM340H-12, Q1 BC817-16W, Q2 BC817-16W

Commit message: Start work on cost reduction, including eliminating SMD componenents (whose S&H were very high)
Parts:
- removed Q1, Q2: BC817-16W, semicon-smd-ipc:NPN-TRANSISTOR_SOT23
- added T1, T2: 2N3565, transistor:2N3565
- F1, F2: value PTCSMD -> PTCPTH; device SparkFun-PowerIC:PTCSMD -> SparkFun-PowerIC:PTCPTH
Connections:
- net GND: now also T2.E; no longer Q2.E
- net N$4: now also T1.E, T2.C; no longer Q1.E, Q2.C
- net N$7: now also T1.C; no longer Q1.C
- net N$8: now also T1.B; no longer Q1.B
- net N$9: now also T2.B; no longer Q2.B
Changed lines of the file:
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@@
 </classes>
 <parts>
-<part name="Q1" library="semicon-smd-ipc" deviceset="NPN-TRANSISTOR_" device="SOT23" value="BC817-16W"/>
-<part name="Q2" library="semicon-smd-ipc" deviceset="NPN-TRANSISTOR_" device="SOT23" value="BC817-16W"/>
 <part name="SG2" library="buzzer" deviceset="F/QMX" device=""/>
 <part name="LED3" library="led" deviceset="TLLY4400" device=""/>
@@
 <part name="D2" library="SparkFun-DiscreteSemi" deviceset="DIODE-ZENER" device="PTH"/>
 <part name="D3" library="SparkFun-DiscreteSemi" deviceset="DIODE-ZENER" device="PTH"/>
-<part name="F1" library="SparkFun-PowerIC" deviceset="PTC" device="SMD"/>
-<part name="F2" library="SparkFun-PowerIC" deviceset="PTC" device="SMD"/>
 <part name="R2" library="SparkFun-Passives" deviceset="RESISTOR" device="PTH-1/2W"/>
 <part name="SUPPLY1" library="SparkFun-Aesthetics" deviceset="VCC" device=""/>
 <part name="GND1" library="SparkFun-Aesthetics" deviceset="GND" device=""/>
+<part name="T1" library="transistor" deviceset="2N3565" device=""/>
+<part name="T2" library="transistor" deviceset="2N3565" device=""/>
+<part name="F1" library="SparkFun-PowerIC" deviceset="PTC" device="PTH"/>
+<part name="F2" library="SparkFun-PowerIC" deviceset="PTC" device="PTH"/>
 </parts>
 <sheets>
@@
 </plain>
 <instances>
-<instance part="Q1" gate="G$1" x="83.82" y="73.66"/>
-<instance part="Q2" gate="G$1" x="83.82" y="58.42"/>
 <instance part="SG2" gate="G$1" x="142.24" y="96.52"/>
 <instance part="LED3" gate="G$1" x="149.86" y="76.2" rot="R90"/>
@@
 <attribute name="NAME" x="71.12" y="55.3974" size="1.778" layer="95" rot="R180"/>
 </instance>
-<instance part="F1" gate="G$1" x="55.88" y="73.66"/>
-<instance part="F2" gate="G$1" x="55.88" y="58.42"/>
 <instance part="R2" gate="G$1" x="142.24" y="76.2"/>
 <instance part="SUPPLY1" gate="G$1" x="22.86" y="55.88"/>
 <instance part="GND1" gate="1" x="22.86" y="50.8"/>
+<instance part="T1" gate="G$1" x="83.82" y="73.66"/>
+<instance part="T2" gate="G$1" x="83.82" y="58.42"/>
+<instance part="F1" gate="G$1" x="55.88" y="73.66"/>
+<instance part="F2" gate="G$1" x="55.88" y="58.42"/>
 </instances>
 <busses>
@@
 <net name="N$4" class="0">
 <segment>
-<pinref part="Q1" gate="G$1" pin="E"/>
-<pinref part="Q2" gate="G$1" pin="C"/>
 <wire x1="86.36" y1="68.58" x2="86.36" y2="63.5" width="0.1524" layer="91"/>
+<pinref part="T1" gate="G$1" pin="E"/>
+<pinref part="T2" gate="G$1" pin="C"/>
 </segment>
 </net>
@@
 <wire x1="48.26" y1="96.52" x2="60.96" y2="96.52" width="0.1524" layer="91"/>
 <junction x="48.26" y="96.52"/>
-<pinref part="Q2" gate="G$1" pin="E"/>
 <wire x1="86.36" y1="53.34" x2="86.36" y2="43.18" width="0.1524" layer="91"/>
 <wire x1="86.36" y1="43.18" x2="71.12" y2="43.18" width="0.1524" layer="91"/>
@@
 <junction x="154.94" y="76.2"/>
 <pinref part="GND1" gate="1" pin="GND"/>
+<pinref part="T2" gate="G$1" pin="E"/>
 </segment>
 </net>
@@
 <segment>
 <pinref part="D1" gate="G$1" pin="C"/>
-<pinref part="Q1" gate="G$1" pin="C"/>
 <wire x1="86.36" y1="88.9" x2="86.36" y2="78.74" width="0.1524" layer="91"/>
+<pinref part="T1" gate="G$1" pin="C"/>
 </segment>
 </net>
 <net name="N$8" class="0">
 <segment>
-<pinref part="Q1" gate="G$1" pin="B"/>
 <pinref part="D2" gate="G$1" pin="C"/>
 <wire x1="71.12" y1="73.66" x2="81.28" y2="73.66" width="0.1524" layer="91"/>
-<pinref part="F1" gate="G$1" pin="2"/>
 <wire x1="63.5" y1="73.66" x2="71.12" y2="73.66" width="0.1524" layer="91"/>
 <junction x="71.12" y="73.66"/>
+<pinref part="T1" gate="G$1" pin="B"/>
+<pinref part="F1" gate="G$1" pin="2"/>
 </segment>
 </net>
 <net name="N$9" class="0">
 <segment>
-<pinref part="Q2" gate="G$1" pin="B"/>
 <pinref part="D3" gate="G$1" pin="C"/>
 <wire x1="66.04" y1="58.42" x2="81.28" y2="58.42" width="0.1524" layer="91"/>
-<pinref part="F2" gate="G$1" pin="2"/>
 <wire x1="63.5" y1="58.42" x2="66.04" y2="58.42" width="0.1524" layer="91"/>
 <junction x="66.04" y="58.42"/>
+<pinref part="T2" gate="G$1" pin="B"/>
+<pinref part="F2" gate="G$1" pin="2"/>
 </segment>
 </net>
@@
 <wire x1="22.86" y1="91.44" x2="33.02" y2="91.44" width="0.1524" layer="91"/>
 <wire x1="33.02" y1="91.44" x2="50.8" y2="73.66" width="0.1524" layer="91"/>
-<pinref part="F1" gate="G$1" pin="1"/>
 <wire x1="22.86" y1="91.44" x2="22.86" y2="88.9" width="0.1524" layer="91"/>
 <wire x1="22.86" y1="73.66" x2="35.56" y2="73.66" width="0.1524" layer="91"/>
 <wire x1="35.56" y1="73.66" x2="50.8" y2="58.42" width="0.1524" layer="91"/>
+<wire x1="22.86" y1="71.12" x2="22.86" y2="73.66" width="0.1524" layer="91"/>
+<pinref part="F1" gate="G$1" pin="1"/>
 <pinref part="F2" gate="G$1" pin="1"/>
-<wire x1="22.86" y1="71.12" x2="22.86" y2="73.66" width="0.1524" layer="91"/>
-</segment>
-</net>
+</segment>
+</net>
