File: eagle/scifair/sci fair schematic.brd (EAGLE design)
At the start: 46.7 x 74.9 mm, 16 parts, among them IC1 LM555N, IC2 LM340H-12, T1 2N3565, T2 2N3565

Commit message: Remove extraneous vias in ground and VCC pours
Routing:
- net GND: track 36.9 -> 35.3 mm, vias 12 -> 6
- net VCC: vias 5 -> 1
Changed lines of the file:
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@@
 <vertex x="69.85" y="16.51"/>
 </polygon>
-<wire x1="87.63" y1="64.77" x2="86.36" y2="66.04" width="0.4064" layer="16"/>
-<wire x1="86.36" y1="66.04" x2="82.55" y2="66.04" width="0.4064" layer="16"/>
 <polygon width="0.4064" layer="16">
 <vertex x="85.09" y="69.85"/>
@@
 <vertex x="85.09" y="67.31"/>
 </polygon>
-<via x="96.52" y="55.88" extent="1-16" drill="0.6" shape="square"/>
 <via x="90.17" y="67.31" extent="1-16" drill="0.6" shape="square"/>
-<via x="86.36" y="68.58" extent="1-16" drill="0.6" shape="square"/>
-<wire x1="96.52" y1="55.88" x2="96.52" y2="60.2488" width="0.4064" layer="16"/>
-<wire x1="86.36" y1="66.04" x2="86.36" y2="68.58" width="0.4064" layer="16"/>
-<via x="72.39" y="63.5" extent="1-16" drill="0.6" shape="square"/>
-<via x="72.39" y="60.96" extent="1-16" drill="0.6" shape="square"/>
-<via x="72.39" y="53.34" extent="1-16" drill="0.6" shape="square"/>
-<via x="72.39" y="49.53" extent="1-16" drill="0.6" shape="square"/>
-<via x="72.39" y="44.45" extent="1-16" drill="0.6" shape="square"/>
-<via x="64.77" y="41.91" extent="1-16" drill="0.6" shape="square"/>
 <polygon width="0.4064" layer="16">
 <vertex x="85.09" y="24.13"/>
@@
 <vertex x="66.04" y="57.15"/>
 <vertex x="64.77" y="55.88"/>
-<vertex x="64.77" y="52.07"/>
 <vertex x="64.77" y="50.8"/>
 <vertex x="66.04" y="49.53"/>
 <vertex x="66.04" y="46.99"/>
-<vertex x="64.77" y="45.72"/>
 <vertex x="63.5" y="44.45"/>
 <vertex x="63.5" y="40.64"/>
@@
 <vertex x="82.55" y="45.72"/>
 <vertex x="83.82" y="44.45"/>
-<vertex x="83.82" y="43.18"/>
-<vertex x="82.55" y="41.91"/>
-<vertex x="81.28" y="41.91"/>
-<vertex x="80.01" y="40.64"/>
+<vertex x="83.82" y="39.37"/>
+<vertex x="80.01" y="39.37"/>
 <vertex x="80.01" y="25.4"/>
 <vertex x="81.28" y="24.13"/>
 </polygon>
-<via x="82.55" y="29.21" extent="1-16" drill="0.6" shape="square"/>
-<wire x1="82.55" y1="29.21" x2="86.36" y2="29.21" width="0.4064" layer="16"/>
-<wire x1="72.39" y1="44.45" x2="76.2" y2="44.45" width="0.4064" layer="16"/>
-<wire x1="72.39" y1="49.53" x2="75.184" y2="49.53" width="0.4064" layer="16"/>
-<wire x1="72.39" y1="53.34" x2="75.184" y2="53.34" width="0.4064" layer="16"/>
-<wire x1="74.93" y1="57.15" x2="74.93" y2="58.42" width="0.4064" layer="16"/>
-<wire x1="74.93" y1="58.42" x2="72.39" y2="60.96" width="0.4064" layer="16"/>
-<wire x1="69.85" y1="63.5" x2="72.39" y2="63.5" width="0.4064" layer="16"/>
 <via x="72.39" y="13.97" extent="1-16" drill="0.6" shape="square"/>
 <polygon width="0.4064" layer="1">
@@
 <vertex x="85.09" y="55.88"/>
 <vertex x="85.09" y="41.91"/>
-<vertex x="82.55" y="39.37"/>
+<vertex x="80.01" y="41.91"/>
+<vertex x="80.01" y="39.37"/>
 <vertex x="76.2" y="39.37"/>
+<vertex x="76.2" y="41.91"/>
 <vertex x="73.66" y="41.91"/>
 <vertex x="73.66" y="55.88"/>
@@
 </polygon>
 <via x="95.25" y="13.97" extent="1-16" drill="0.6" shape="square"/>
-<wire x1="64.77" y1="38.1" x2="64.77" y2="41.91" width="0.4064" layer="16"/>
 <polygon width="0.4064" layer="1">
 <vertex x="80.01" y="3.81"/>
@@
 <vertex x="80.01" y="15.24"/>
 </polygon>
+<wire x1="69.85" y1="63.5" x2="72.39" y2="63.5" width="0.4064" layer="16"/>
+<wire x1="75.184" y1="49.53" x2="72.39" y2="49.53" width="0.4064" layer="16"/>
+<wire x1="75.184" y1="53.34" x2="72.39" y2="53.34" width="0.4064" layer="16"/>
+<wire x1="64.77" y1="38.1" x2="64.77" y2="41.91" width="0.4064" layer="16"/>
+<wire x1="76.2" y1="44.45" x2="76.2" y2="45.72" width="0.4064" layer="16"/>
+<wire x1="76.2" y1="44.45" x2="72.39" y2="44.45" width="0.4064" layer="16"/>
+<wire x1="86.36" y1="29.21" x2="83.82" y2="29.21" width="0.4064" layer="16"/>
+<via x="82.55" y="38.1" extent="1-16" drill="0.6" shape="square"/>
+<wire x1="82.55" y1="66.04" x2="86.36" y2="66.04" width="0.4064" layer="16"/>
+<wire x1="86.36" y1="66.04" x2="87.63" y2="64.77" width="0.4064" layer="16"/>
+<wire x1="87.63" y1="64.77" x2="87.63" y2="67.31" width="0.4064" layer="16"/>
+<via x="69.85" y="50.8" extent="1-16" drill="0.6" shape="square"/>
+<wire x1="74.93" y1="57.15" x2="72.39" y2="59.69" width="0.4064" layer="16"/>
+<via x="96.52" y="55.88" extent="1-16" drill="0.6" shape="square"/>
+<wire x1="96.52" y1="60.2488" x2="93.2688" y2="60.2488" width="0.4064" layer="16"/>
+<wire x1="93.2688" y1="60.2488" x2="92.71" y2="59.69" width="0.4064" layer="16"/>
 </signal>
 <signal name="5V">
@@
 <vertex x="73.66" y="41.91"/>
 </polygon>
-<via x="81.28" y="17.78" extent="1-16" drill="0.6" shape="square"/>
-<via x="90.17" y="17.78" extent="1-16" drill="0.6" shape="square"/>
-<wire x1="81.28" y1="17.78" x2="81.28" y2="21.59" width="0.4064" layer="16"/>
-<wire x1="90.17" y1="17.78" x2="90.17" y2="21.59" width="0.4064" layer="16"/>
 <via x="95.25" y="17.78" extent="1-16" drill="0.6" shape="square"/>
-<via x="72.39" y="38.1" extent="1-16" drill="0.6" shape="square"/>
-<wire x1="72.39" y1="38.1" x2="67.31" y2="38.1" width="0.4064" layer="16"/>
-<via x="77.47" y="40.64" extent="1-16" drill="0.6" shape="square"/>
-<wire x1="77.47" y1="40.64" x2="81.28" y2="44.45" width="0.4064" layer="16"/>
+<wire x1="67.31" y1="38.1" x2="72.39" y2="38.1" width="0.4064" layer="16"/>
+<wire x1="81.28" y1="44.45" x2="77.47" y2="40.64" width="0.4064" layer="16"/>
+<wire x1="81.28" y1="21.59" x2="81.28" y2="17.78" width="0.4064" layer="16"/>
+<wire x1="90.17" y1="21.59" x2="90.17" y2="17.78" width="0.4064" layer="16"/>
 </signal>
 <signal name="N$4">
